File: Schematic/robot/robot.sch (KiCad schematic (older format))
At the start: 8 parts, among them U1 L298HN

Commit message: Documentation
Parts:
- added SW?: SW_MEC_5E, symbol Switch:SW_MEC_5E
- R1, R4: value R -> 10k
- R2, R3: value R -> 330
Connections:
- net GND: now also SW?.3 (K), SW?.4 (A)
- new net PIN_2: SW?.1, SW?.2
Other:
- moved on the sheet: A1, R1, R2, R3, R4, S1, S2, U1
Changed lines of the file:
@@
 L MCU_Module:Arduino_UNO_R3 A1
 U 1 1 5F8E5CBD
-P 2750 2400
-F 0 "A1" H 2750 3581 50  0000 C CNN
-F 1 "Arduino_UNO_R3" H 2750 3490 50  0000 C CNN
-F 2 "Module:Arduino_UNO_R3" H 2750 2400 50  0001 C CIN
-F 3 "https://www.arduino.cc/en/Main/arduinoBoardUno" H 2750 2400 50  0001 C CNN
-	1    2750 2400
+P 4000 3300
+F 0 "A1" H 4000 4481 50  0000 C CNN
+F 1 "Arduino_UNO_R3" H 4000 4390 50  0000 C CNN
+F 2 "Module:Arduino_UNO_R3" H 4000 3300 50  0001 C CIN
+F 3 "https://www.arduino.cc/en/Main/arduinoBoardUno" H 4000 3300 50  0001 C CNN
+	1    4000 3300
 	1    0    0    -1
 $EndComp
@@
 L OPB620:OPB620 S2
 U 1 1 5F8E7D7F
-P 5900 1750
-F 0 "S2" H 5850 2120 50  0000 C CNN
-F 1 "OPB620" H 5850 2029 50  0000 C CNN
-F 2 "Schematic:OPTO_OPB620" H 5900 1750 50  0001 L BNN
-F 3 "Optex" H 5900 1750 50  0001 L BNN
-	1    5900 1750
+P 7150 2650
+F 0 "S2" H 7100 3020 50  0000 C CNN
+F 1 "OPB620" H 7100 2929 50  0000 C CNN
+F 2 "Schematic:OPTO_OPB620" H 7150 2650 50  0001 L BNN
+F 3 "Optex" H 7150 2650 50  0001 L BNN
+	1    7150 2650
 	1    0    0    -1
 $EndComp
@@
 L Device:R R1
 U 1 1 5F8EBF51
-P 4800 1300
-F 0 "R1" H 4870 1346 50  0000 L CNN
-F 1 "R" H 4870 1255 50  0000 L CNN
-F 2 "Resistor_THT:R_Axial_DIN0207_L6.3mm_D2.5mm_P10.16mm_Horizontal" V 4730 1300 50  0001 C CNN
-F 3 "~" H 4800 1300 50  0001 C CNN
-	1    4800 1300
+P 6050 2200
+F 0 "R1" H 6120 2246 50  0000 L CNN
+F 1 "10k" H 6120 2155 50  0000 L CNN
+F 2 "Resistor_THT:R_Axial_DIN0207_L6.3mm_D2.5mm_P10.16mm_Horizontal" V 5980 2200 50  0001 C CNN
+F 3 "~" H 6050 2200 50  0001 C CNN
+	1    6050 2200
 	1    0    0    -1
 $EndComp
@@
 L Device:R R4
 U 1 1 5F8EF4E7
-P 6250 1150
-F 0 "R4" H 6320 1196 50  0000 L CNN
-F 1 "R" H 6320 1105 50  0000 L CNN
-F 2 "Resistor_THT:R_Axial_DIN0207_L6.3mm_D2.5mm_P10.16mm_Horizontal" V 6180 1150 50  0001 C CNN
-F 3 "~" H 6250 1150 50  0001 C CNN
-	1    6250 1150
+P 7500 2050
+F 0 "R4" H 7570 2096 50  0000 L CNN
+F 1 "10k" H 7570 2005 50  0000 L CNN
+F 2 "Resistor_THT:R_Axial_DIN0207_L6.3mm_D2.5mm_P10.16mm_Horizontal" V 7430 2050 50  0001 C CNN
+F 3 "~" H 7500 2050 50  0001 C CNN
+	1    7500 2050
 	1    0    0    -1
 $EndComp
@@
 L Device:R R2
 U 1 1 5F8F058A
-P 3750 1800
-F 0 "R2" V 3957 1800 50  0000 C CNN
-F 1 "R" V 3866 1800 50  0000 C CNN
-F 2 "Resistor_THT:R_Axial_DIN0207_L6.3mm_D2.5mm_P10.16mm_Horizontal" V 3680 1800 50  0001 C CNN
-F 3 "~" H 3750 1800 50  0001 C CNN
-	1    3750 1800
+P 5000 2700
+F 0 "R2" V 5207 2700 50  0000 C CNN
+F 1 "330" V 5116 2700 50  0000 C CNN
+F 2 "Resistor_THT:R_Axial_DIN0207_L6.3mm_D2.5mm_P10.16mm_Horizontal" V 4930 2700 50  0001 C CNN
+F 3 "~" H 5000 2700 50  0001 C CNN
+	1    5000 2700
 	0    -1   -1   0
 $EndComp
@@
 L Device:R R3
 U 1 1 5F8F0A1B
-P 5200 1850
-F 0 "R3" V 4993 1850 50  0000 C CNN
-F 1 "R" V 5084 1850 50  0000 C CNN
-F 2 "Resistor_THT:R_Axial_DIN0207_L6.3mm_D2.5mm_P10.16mm_Horizontal" V 5130 1850 50  0001 C CNN
-F 3 "~" H 5200 1850 50  0001 C CNN
-	1    5200 1850
+P 6450 2750
+F 0 "R3" V 6243 2750 50  0000 C CNN
+F 1 "330" V 6334 2750 50  0000 C CNN
+F 2 "Resistor_THT:R_Axial_DIN0207_L6.3mm_D2.5mm_P10.16mm_Horizontal" V 6380 2750 50  0001 C CNN
+F 3 "~" H 6450 2750 50  0001 C CNN
+	1    6450 2750
 	0    1    1    0
 $EndComp
@@
 L Driver_Motor:L298HN U1
 U 1 1 5F8F49D9
-P 5400 3200
-F 0 "U1" H 5400 4081 50  0000 C CNN
-F 1 "L298HN" H 5400 3990 50  0000 C CNN
-F 2 "Package_TO_SOT_THT:TO-220-15_P2.54x2.54mm_StaggerOdd_Lead4.58mm_Vertical" H 5450 2550 50  0001 L CNN
-F 3 "http://www.st.com/st-web-ui/static/active/en/resource/technical/document/datasheet/CD00000240.pdf" H 5550 3450 50  0001 C CNN
-	1    5400 3200
+P 6650 4100
+F 0 "U1" H 6650 4981 50  0000 C CNN
+F 1 "L298HN" H 6650 4890 50  0000 C CNN
+F 2 "Package_TO_SOT_THT:TO-220-15_P2.54x2.54mm_StaggerOdd_Lead4.58mm_Vertical" H 6700 3450 50  0001 L CNN
+F 3 "http://www.st.com/st-web-ui/static/active/en/resource/technical/document/datasheet/CD00000240.pdf" H 6800 4350 50  0001 C CNN
+	1    6650 4100
 	1    0    0    -1
 $EndComp
@@
 L OPB620:OPB620 S1
 U 1 1 5F8E73E2
-P 4500 1700
-F 0 "S1" H 4450 2070 50  0000 C CNN
-F 1 "OPB620" H 4450 1979 50  0000 C CNN
-F 2 "Schematic:OPTO_OPB620" H 4500 1700 50  0001 L BNN
-F 3 "Optex" H 4500 1700 50  0001 L BNN
-	1    4500 1700
-	1    0    0    -1
-$EndComp
-Wire Wire Line
-	2950 1400 3350 1400
-Wire Wire Line
-	3600 1400 3600 1800
-Wire Wire Line
-	3900 1800 4100 1800
-Wire Wire Line
-	4800 1450 4800 1500
-Wire Wire Line
-	4800 1150 4650 1150
-Wire Wire Line
-	3600 1150 3600 1400
-Connection ~ 3600 1400
-Text GLabel 2750 3500 3    50   Input ~ 0
-GND
-Text GLabel 4100 1600 0    50   Input ~ 0
-GND
-Text GLabel 4800 1800 3    50   Input ~ 0
-GND
-Text GLabel 4900 1500 2    50   Input ~ 0
+P 5750 2600
+F 0 "S1" H 5700 2970 50  0000 C CNN
+F 1 "OPB620" H 5700 2879 50  0000 C CNN
+F 2 "Schematic:OPTO_OPB620" H 5750 2600 50  0001 L BNN
+F 3 "Optex" H 5750 2600 50  0001 L BNN
+	1    5750 2600
+	1    0    0    -1
+$EndComp
+Wire Wire Line
+	4200 2300 4600 2300
+Wire Wire Line
+	4850 2300 4850 2700
+Wire Wire Line
+	5150 2700 5350 2700
+Wire Wire Line
+	6050 2350 6050 2400
+Wire Wire Line
+	6050 2050 5900 2050
+Wire Wire Line
+	4850 2050 4850 2300
+Connection ~ 4850 2300
+Text GLabel 4000 4400 3    50   Input ~ 0
+GND
+Text GLabel 5350 2500 0    50   Input ~ 0
+GND
+Text GLabel 6050 2700 3    50   Input ~ 0
+GND
+Text GLabel 6150 2400 2    50   Input ~ 0
 PIN_8
 Wire Wire Line
-	4900 1500 4800 1500
-Connection ~ 4800 1500
-Wire Wire Line
-	4800 1500 4800 1600
-Text GLabel 2000 2600 0    50   Input ~ 0
+	6150 2400 6050 2400
+Connection ~ 6050 2400
+Wire Wire Line
+	6050 2400 6050 2500
+Text GLabel 3250 3500 0    50   Input ~ 0
 PIN_8
 Wire Wire Line
-	3600 1800 3600 2250
-Wire Wire Line
-	3600 2250 5050 2250
-Wire Wire Line
-	5050 2250 5050 1850
-Connection ~ 3600 1800
-Wire Wire Line
-	5350 1850 5500 1850
-Wire Wire Line
-	6200 1650 6250 1650
-Wire Wire Line
-	6250 1650 6250 1450
-Wire Wire Line
-	6250 1000 4650 1000
-Wire Wire Line
-	4650 1000 4650 1150
-Connection ~ 4650 1150
-Wire Wire Line
-	4650 1150 3600 1150
-Text GLabel 6200 1850 3    50   Input ~ 0
-GND
-Text GLabel 5500 1650 1    50   Input ~ 0
-GND
-Text GLabel 6400 1450 2    50   Input ~ 0
+	4850 2700 4850 3150
+Wire Wire Line
+	4850 3150 6300 3150
+Wire Wire Line
+	6300 3150 6300 2750
+Connection ~ 4850 2700
+Wire Wire Line
+	6600 2750 6750 2750
+Wire Wire Line
+	7450 2550 7500 2550
+Wire Wire Line
+	7500 2550 7500 2350
+Wire Wire Line
+	7500 1900 5900 1900
+Wire Wire Line
+	5900 1900 5900 2050
+Connection ~ 5900 2050
+Wire Wire Line
+	5900 2050 4850 2050
+Text GLabel 7450 2750 3    50   Input ~ 0
+GND
+Text GLabel 6750 2550 1    50   Input ~ 0
+GND
+Text GLabel 7650 2350 2    50   Input ~ 0
 PIN_7
 Wire Wire Line
-	6400 1450 6250 1450
-Connection ~ 6250 1450
-Wire Wire Line
-	6250 1450 6250 1300
-Text GLabel 2000 2500 0    50   Input ~ 0
+	7650 2350 7500 2350
+Connection ~ 7500 2350
+Wire Wire Line
+	7500 2350 7500 2200
+Text GLabel 3250 3400 0    50   Input ~ 0
 PIN_7
 Wire Wire Line
-	2000 2500 2250 2500
-Wire Wire Line
-	2000 2600 2250 2600
-Text GLabel 4800 2700 0    50   Input ~ 0
+	3250 3400 3500 3400
+Wire Wire Line
+	3250 3500 3500 3500
+Text GLabel 6050 3600 0    50   Input ~ 0
 PIN_9
-Text GLabel 4800 2800 0    50   Input ~ 0
+Text GLabel 6050 3700 0    50   Input ~ 0
 PIN_10
-Text GLabel 4800 3100 0    50   Input ~ 0
+Text GLabel 6050 4000 0    50   Input ~ 0
 PIN_5
-Text GLabel 4800 3200 0    50   Input ~ 0
+Text GLabel 6050 4100 0    50   Input ~ 0
 PIN_6
-Text GLabel 2000 2700 0    50   Input ~ 0
+Text GLabel 3250 3600 0    50   Input ~ 0
 PIN_9
-Text GLabel 2050 2800 0    50   Input ~ 0
+Text GLabel 3300 3700 0    50   Input ~ 0
 PIN_10
-Text GLabel 2000 2300 0    50   Input ~ 0
+Text GLabel 3250 3200 0    50   Input ~ 0
 PIN_5
-Text GLabel 2000 2400 0    50   Input ~ 0
+Text GLabel 3250 3300 0    50   Input ~ 0
 PIN_6
 Wire Wire Line
-	2000 2700 2250 2700
-Wire Wire Line
-	2050 2800 2250 2800
-Wire Wire Line
-	2000 2300 2250 2300
-Wire Wire Line
-	2000 2400 2250 2400
-Wire Wire Line
-	2850 3500 2850 4050
-Wire Wire Line
-	2850 4050 5400 4050
-Wire Wire Line
-	5400 4050 5400 3900
-Wire Wire Line
-	3350 1400 3350 2300
-Wire Wire Line
-	3350 2300 5500 2300
-Wire Wire Line
-	5500 2300 5500 2500
-Connection ~ 3350 1400
-Wire Wire Line
-	3350 1400 3600 1400
-Text GLabel 5400 2500 0    50   Input ~ 0
+	3250 3600 3500 3600
+Wire Wire Line
+	3300 3700 3500 3700
+Wire Wire Line
+	3250 3200 3500 3200
+Wire Wire Line
+	3250 3300 3500 3300
+Wire Wire Line
+	4100 4400 4100 4950
+Wire Wire Line
+	4100 4950 6650 4950
+Wire Wire Line
+	6650 4950 6650 4800
+Wire Wire Line
+	4600 2300 4600 3200
+Wire Wire Line
+	4600 3200 6750 3200
+Wire Wire Line
+	6750 3200 6750 3400
+Connection ~ 4600 2300
+Wire Wire Line
+	4600 2300 4850 2300
+Text GLabel 6650 3400 0    50   Input ~ 0
 VIN
-Text GLabel 2650 1400 0    50   Input ~ 0
+Text GLabel 3900 2300 0    50   Input ~ 0
 VIN
+$Comp
+L Switch:SW_MEC_5E SW?
+U 1 1 5F90EC23
+P 9350 3200
+F 0 "SW?" H 9350 3585 50  0000 C CNN
+F 1 "SW_MEC_5E" H 9350 3494 50  0000 C CNN
+F 2 "" H 9350 3500 50  0001 C CNN
+F 3 "http://www.apem.com/int/index.php?controller=attachment&id_attachment=1371" H 9350 3500 50  0001 C CNN
+	1    9350 3200
+	1    0    0    -1
+$EndComp
+Wire Wire Line
+	9150 3100 9150 3200
+Wire Wire Line
+	9550 3100 9550 3200
+Text GLabel 9100 3300 0    50   Input ~ 0
+PIN_2
+Text GLabel 9650 3350 2    50   Input ~ 0
+GND
+Wire Wire Line
+	9100 3300 9100 3100
+Wire Wire Line
+	9100 3100 9150 3100
+Connection ~ 9150 3100
+Wire Wire Line
+	9550 3100 9650 3100
+Wire Wire Line
+	9650 3100 9650 3350
+Connection ~ 9550 3100
 $EndSCHEMATC
